Commit message: success

File: raisim_gym/env/env/jueying/jueying/jueying_raisim.xacro (robot description, xacro)
@@ -32,6 +32,6 @@
     <xacro:property name="motor_torque" value="0.0"/>
     <xacro:property name="motor_vec" value="0.0"/>
-    <xacro:property name="motor_damp" value="1.2"/>
-    <xacro:property name="motor_fric" value="0.1"/>
+    <xacro:property name="motor_damp" value="0.0"/>
+    <xacro:property name="motor_fric" value="0.0"/>
     <xacro:property name="PI" value="3.14159265359"/>
     <xacro:property name="sx_l" value="0.204"/>
@@ -46,8 +46,9 @@
     <xacro:property name="sk_x" value="0.028"/>
     <xacro:property name="sk_r" value="0.0305"/>
+    <xacro:property name="mass_ratio" value ="0.3" />
     <link name="origin_link">
     </link>
     <joint name="origin_baselink_joint" type="fixed">
-        <origin xyz="0 0 0.6" rpy="0 0 0"/>
+        <origin xyz="0 0 0.2" rpy="0 0 0"/>
         <parent link="origin_link"/>
         <child link="base_link"/>
@@ -56,5 +57,5 @@
         <inertial>
             <origin xyz="0.0030652 0.0043949 0.015248" rpy="0 0 0" />
-            <mass value="30.0" />
+            <mass value="${mass_ratio*30.0}" />
             <inertia ixx="0.15234" ixy="0.00092094" ixz="-0.0095582" iyy="0.68188" iyz="0.00091552" izz="0.64094" />
         </inertial>
@@ -62,5 +63,5 @@
             <origin xyz="0 0 0" rpy="0 0 0" />
             <geometry>
-                <mesh filename="package://jueying_description/meshes/base_link.STL" />
+                <mesh filename="meshes/base_link.STL" />
             </geometry>
             <material name="white"/>
@@ -89,5 +90,5 @@
             <inertial>
                 <origin xyz="0.0 ${is_l*0.038} 0.0" rpy="0 0 0" />
-                <mass value="3.0" />
+                <mass value="${mass_ratio*3.0}" />
                 <inertia ixx="0.00084975" ixy="2.5128E-05" ixz="-3.1095E-05" iyy="0.0016235" iyz="1.9684E-05" izz="0.0012084" />
             </inertial>
@@ -95,5 +96,5 @@
                 <origin xyz="0 0 0" rpy="0 0 0" />
                 <geometry>
-                    <mesh filename="package://jueying_description/meshes/${name}_HipX.STL" />
+                    <mesh filename="meshes/${name}_HipX.STL" />
                 </geometry>
                 <material name="white"/>
@@ -111,5 +112,5 @@
             <child link="${name}_HipX" />
             <axis xyz="1 0 0" />
-            <limit lower="-0.39" upper="0.39" effort="37.8" velocity="13.6" />
+            <limit lower="-0.39" upper="0.39" effort="37.8" velocity="33.6" />
             <dynamics damping="${motor_damp}" friction="${motor_fric}" />
         </joint>
@@ -117,5 +118,5 @@
             <inertial>
                 <origin xyz="0.0 ${is_l*0.026983} -0.047138" rpy="0 0 0" />
-                <mass value="6.0" />
+                <mass value="${mass_ratio*6.0}" />
                 <inertia ixx="0.0091835" ixy="-5.5596E-05" ixz="-0.00026799" iyy="0.0095232" iyz="-0.0011185" izz="0.0023439" />
             </inertial>
@@ -123,5 +124,5 @@
                 <origin xyz="0 0 0" rpy="0 0 0" />
                 <geometry>
-                    <mesh filename="package://jueying_description/meshes/${name}_HipY.STL" />
+                    <mesh filename="meshes/${name}_HipY.STL" />
                 </geometry>
                 <material name="white"/>
@@ -144,6 +145,6 @@
             <parent link="${name}_HipX" />
             <child link="${name}_HipY" />
-            <axis xyz="0 -1 0" />
-            <limit lower="-2.27" upper="0.18" effort="58.3" velocity="13.4" />
+            <axis xyz="0 1 0" />
+            <limit upper="2.27" lower="-0.18" effort="38.3" velocity="33.4" />
             <dynamics damping="${motor_damp}" friction="${motor_fric}" />
         </joint>
@@ -151,5 +152,5 @@
             <inertial>
                 <origin xyz="0.0 0.0 -0.14462" rpy="0 0 0" />
-                <mass value="1.0" />
+                <mass value="${mass_ratio*1.0}" />
                 <inertia ixx="0.0048214" ixy="-9.1437E-08" ixz="8.5221E-05" iyy="0.0048402" iyz="1.3168E-06" izz="5.8603E-05" />
             </inertial>
@@ -157,5 +158,5 @@
                 <origin xyz="0 0 0" rpy="0 0 0" />
                 <geometry>
-                    <mesh filename="package://jueying_description/meshes/${name}_Knee.STL" />
+                    <mesh filename="meshes/${name}_Knee.STL" />
                 </geometry>
                 <material name="white"/>
@@ -178,6 +179,6 @@
             <parent link="${name}_HipY" />
             <child link="${name}_Knee" />
-            <axis xyz="0 -1 0" />
-            <limit lower="0.66" upper="2.73" effort="58.3" velocity="13.4" />
+            <axis xyz="0 1 0" />
+            <limit upper="-0.66" lower="-2.73" effort="38.3" velocity="33.4" />
             <dynamics damping="${motor_damp}" friction="${motor_fric}" />
         </joint>
